File: uTari_kicad/uTari_kicad.kicad_pcb (KiCad board)
At the start: 4 copper layers, 180 x 90 mm, 98 parts, among them J1 Conn_01x02_Pin, J2 L Joystick, J3 R Joystick, J4 Audio Out, J5 Video Out, J6 Cartridge Port, J7 Conn_01x03, J8 Conn_01x03, Q1 2N3906, Q2 2N3904, SW1 SW_SPDT, SW2 R Diff, SW3 L Diff, SW4 SW_SPDT, SW5 Select, SW6 Reset, U1 6507, U2 TIA C010444, U3 RIOT, U4 L7805, Y1 3.579545 MHz

Commit message: Save PCB progress.
Parts:
- added J9: GND, Connector_PinSocket_2.54mm:PinSocket_1x02_P2.54mm_Vertical, F.Cu at (329.5, 161.7)
- J2: value L Joystick -> L Joy
- J3: value R Joystick -> R Joy
- J4: value Audio Out -> A Out
- J5: value Video Out -> V Out
- SW1, SW2, SW3, SW4: footprint Button_Switch_THT:SW_Slide-03_Wuerth-WS-SLTV_10x2.5x6.4_P2.54mm -> Connector_PinHeader_2.54mm:PinHeader_1x03_P2.54mm_Vertical
- moved R9 270.7 mm to (344.4, 205.3)
- moved R8 267.5 mm to (341.2, 200.7)
- moved R13 245.7 mm to (328.0, 215.6), turned to 90 degrees
- moved R12 244.3 mm to (327.7, 200.7), turned to 180 degrees
- moved R15 240.7 mm to (325.2, 193.8), turned to 180 degrees
- moved R10 238.0 mm to (320.1, 203.8)
- moved R14 237.6 mm to (322.1, 184.6), turned to 180 degrees
- moved R20 234.5 mm to (322.5, 228.0)
- moved R19 233.2 mm to (316.8, 227.0), turned to -90 degrees
- moved R16 233.1 mm to (317.6, 190.8)
- moved R17 232.1 mm to (316.4, 207.2), turned to -90 degrees
- moved R18 230.5 mm to (314.9, 197.9), turned to 90 degrees
- moved R21 229.7 mm to (319.9, 222.4), turned to -90 degrees
- moved R29 229.6 mm to (322.5, 231.0)
- moved R28 227.6 mm to (319.4, 234.1)
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- renumbered C8 to 0.1
Other:
- board size 180 x 90 mm -> 161.6 x 90 mm
- board text added: ".068 Poly"
- board text added: "1"
- board text added: "1N914"
- board text added: "2"
- board text added: "23"
- board text added: "24"
- board text added: "9V"
- board text added: "A"
- board text added: "B"
- board text added: "B&W"
- board text added: "Cartridge Port"
- board text added: "Color"
- board text added: "Color Adjust"
- board text added: "G"
- board text added: "GND"
- board text added: "On"

Commit message: Save PCB progress.
Parts:
- moved R23 43.1 mm to (286.5, 192.0), turned to 0 degrees
- moved R9 41.0 mm to (303.4, 204.9)
- moved J4 34.6 mm to (287.4, 161.6)
- moved J5 34.6 mm to (291.1, 161.6)
- moved J9 34.6 mm to (294.8, 161.6)
- moved R11 34.6 mm to (276.9, 161.6)
- moved R8 32.6 mm to (310.5, 189.6), turned to -90 degrees
- moved C7 31.8 mm to (241.4, 245.3)
- moved U1 31.8 mm to (241.5, 241.1)
- moved R1 31.8 mm to (237.7, 228.4)
- moved C31 31.6 mm to (278.6, 169.2)
- moved D5 31.6 mm to (281.4, 219.3)
- moved R27 31.6 mm to (300.8, 232.8)
- moved RV1 31.6 mm to (291.6, 207.6)
- moved C32 31.6 mm to (298.8, 199.9)
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Other:
- board size 161.6 x 90 mm -> 120.3 x 90 mm
- board text added: "Have you played µTari today?"
- board text added: "µTari v1.0 August 2026 Designed by Nick Bild github.com/nickbild/uTari"

Commit message: PCB complete.
Parts:
- C36: value 22 pF -> 22pF
- C37: value 150 pF -> 150pF
- D2, D3, D4: value 1N914 -> 914
- J4: value A Out -> Audio Out
- J5: value V Out -> Video Out
Routing:
- net Net-(J6-Pin_4): track 0.00 -> 184.5 mm, vias 0 -> 7
- net Net-(D3-K): track 0.00 -> 184.0 mm
- net Net-(SW1-C): track 0.00 -> 161.5 mm
- net Net-(J6-Pin_6): track 0.00 -> 149.2 mm, vias 0 -> 4
- net Net-(J6-Pin_3): track 0.00 -> 143.5 mm, vias 0 -> 1
- net Net-(J6-Pin_15): track 0.00 -> 141.9 mm, vias 0 -> 4
- net Net-(J6-Pin_11): track 0.00 -> 140.7 mm, vias 0 -> 3
- net Net-(J6-Pin_13): track 0.00 -> 140.2 mm, vias 0 -> 3
- net Net-(J6-Pin_5): track 0.00 -> 139.0 mm, vias 0 -> 2
- net Net-(J6-Pin_21): track 0.00 -> 138.5 mm, vias 0 -> 5
- net Net-(J6-Pin_7): track 0.00 -> 137.3 mm, vias 0 -> 4
- net Net-(J6-Pin_8): track 0.00 -> 126.8 mm, vias 0 -> 4
- net Net-(J6-Pin_14): track 0.00 -> 119.2 mm, vias 0 -> 5
- net Net-(J6-Pin_1): track 0.00 -> 118.4 mm, vias 0 -> 2
- net Net-(J6-Pin_9): track 0.00 -> 117.3 mm, vias 0 -> 3
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Other:
- board text added: "914"
- board text removed: "1N914"

Commit message: Minor board updates.
Parts:
- R27: value 2.2K -> 3.3K
- R28: value 1.6K -> 2.2K
- SW5: value Select -> Reset
- SW6: value Reset -> Select
Changed lines of the file:
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@@
 			(plot_on_all_layers_selection 0x00000000_00000000_00000000_00000000)
 			(disableapertmacros no)
-			(usegerberextensions no)
+			(usegerberextensions yes)
 			(usegerberattributes yes)
 			(usegerberadvancedattributes yes)
@@
 			(outputformat 1)
 			(mirror no)
-			(drillshape 1)
+			(drillshape 0)
 			(scaleselection 1)
-			(outputdirectory "")
+			(outputdirectory "gerber/")
 		)
 	)
@@
 			)
 		)
-		(property "Value" "1.6K"
+		(property "Value" "2.2K"
 			(at 3.81 0 0)
 			(layer "F.SilkS")
@@
 			)
 		)
-		(property "Value" "2.2K"
+		(property "Value" "3.3K"
 			(at 7.62 0 0)
 			(layer "F.SilkS")
@@
 			)
 		)
-		(property "Value" "Reset"
+		(property "Value" "Select"
 			(at 3.2004 6.7352 0)
 			(layer "F.SilkS")
@@
 			)
 		)
-		(property "Value" "Select"
+		(property "Value" "Reset"
 			(at 3.1472 6.7352 0)
 			(layer "F.SilkS")
