File: uTari_kicad/uTari_kicad.kicad_sch (KiCad schematic)
At the start: 94 parts, among them J1 Conn_01x02_Pin, J2 L Joystick, J3 R Joystick, J4 Audio Out, J5 Video Out, J6 Cartridge Port, Q1 2N3906, Q2 2N3904, SW1 SW_SPDT, SW2 R Diff, SW3 L Diff, SW4 SW_SPDT, SW5 Select, SW6 Reset, U1 6507, U2 TIA C010444, U3 RIOT, U4 L7805, Y1 3.579545 MHz

Commit message: Save PCB progress.
Parts:
- added J7, J8: Conn_01x03, Connector_PinSocket_2.54mm:PinSocket_1x03_P2.54mm_Vertical, symbol Connector_Generic:Conn_01x03
- added RV2: Brightness, Potentiometer_THT:Potentiometer_ACP_CA6-H2,5_Horizontal, symbol Device:R_Potentiometer_US
- added RV3: Contrast, Potentiometer_THT:Potentiometer_ACP_CA6-H2,5_Horizontal, symbol Device:R_Potentiometer_US
- C1, C10, C11, C12, C13, C14, C15, C16, C17, C18, C19, C20, C21, C22, C23, C24, C29, C30, C32, C33, C34, C35, C36, C37, C4, C5, C6, C8, C9: footprint (none) -> Capacitor_THT:C_Disc_D5.0mm_W2.5mm_P5.00mm
- C2: footprint (none) -> Capacitor_THT:C_Radial_D16.0mm_H31.5mm_P7.50mm
- C25, C26, C27, C28: footprint (none) -> Capacitor_THT:C_Disc_D8.0mm_W5.0mm_P7.50mm
- C3, C31: footprint (none) -> Capacitor_THT:C_Disc_D11.0mm_W5.0mm_P10.00mm
- C7: footprint (none) -> Capacitor_THT:CP_Radial_D5.0mm_P2.50mm
- D1: footprint Diode_THT:D_DO-41_SOD81_P10.16mm_Horizontal -> Diode_THT:D_DO-35_SOD27_P7.62mm_Horizontal
- FB1, FB2, FB3, R10, R11, R12, R13, R14, R15, R16, R17, R18, R19, R2, R20, R21, R22, R23, R25, R26, R28, R29, R4, R5, R6, R7, R8, R9: footprint (none) -> Resistor_THT:R_Axial_DIN0207_L6.3mm_D2.5mm_P7.62mm_Horizontal
- J1: footprint (none) -> Connector_PinSocket_2.54mm:PinSocket_1x02_P2.54mm_Vertical
- J2, J3: footprint (none) -> Connector_PinSocket_2.54mm:PinSocket_1x09_P2.54mm_Vertical
- J4, J5: footprint (none) -> Connector_PinSocket_2.54mm:PinSocket_1x01_P2.54mm_Vertical
- J6: footprint (none) -> Connector_PinSocket_2.54mm:PinSocket_2x12_P2.54mm_Vertical
- R1, R24, R3: footprint (none) -> Resistor_THT:R_Axial_DIN0309_L9.0mm_D3.2mm_P12.70mm_Horizontal
- R27: footprint (none) -> Resistor_THT:R_Axial_DIN0414_L11.9mm_D4.5mm_P15.24mm_Horizontal
- RV1: footprint (none) -> Potentiometer_THT:Potentiometer_ACP_CA6-H2,5_Horizontal
- SW1, SW2, SW3, SW4: footprint (none) -> Button_Switch_THT:SW_Slide-03_Wuerth-WS-SLTV_10x2.5x6.4_P2.54mm
- SW5, SW6: footprint (none) -> Button_Switch_THT:SW_PUSH_6mm
- U4: footprint (none) -> Package_TO_SOT_THT:TO-220-3_Horizontal_TabDown
- Y1: footprint (none) -> Crystal:Resonator-2Pin_W10.0mm_H5.0mm
Connections:
- new net: J8.1 (Pin_1), RV2.1
- new net: J8.2 (Pin_2), RV2.2
- new net: J8.3 (Pin_3), RV2.3
- new net: J7.1 (Pin_1), RV3.1
- new net: J7.2 (Pin_2), RV3.2
- new net: J7.3 (Pin_3), RV3.3
- no-connect marks 5 -> 9

Commit message: Save PCB progress.
Parts:
- added J9: Ground Out, Connector_PinSocket_2.54mm:PinSocket_1x02_P2.54mm_Vertical, symbol Connector:Conn_01x02_Pin
- SW1, SW2, SW3, SW4: footprint Button_Switch_THT:SW_Slide-03_Wuerth-WS-SLTV_10x2.5x6.4_P2.54mm -> Connector_PinHeader_2.54mm:PinHeader_1x03_P2.54mm_Vertical
Connections:
- net GND: now also J9.1 (Pin_1), J9.2 (Pin_2)
Changed lines of the file:
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@@
 			)
 		)
-		(property "Footprint" "Button_Switch_THT:SW_Slide-03_Wuerth-WS-SLTV_10x2.5x6.4_P2.54mm"
+		(property "Footprint" "Connector_PinHeader_2.54mm:PinHeader_1x03_P2.54mm_Vertical"
 			(at 39.37 308.61 0)
 			(hide yes)
@@
 	(symbol
 		(lib_id "power:GND")
+		(at 751.84 135.89 90)
+		(unit 1)
+		(body_style 1)
+		(exclude_from_sim no)
+		(in_bom yes)
+		(on_board yes)
+		(in_pos_files yes)
+		(dnp no)
+		(fields_autoplaced yes)
+		(property "Reference" "#PWR01"
+			(at 758.19 135.89 0)
+			(hide yes)
+			(show_name no)
+			(do_not_autoplace no)
+			(effects
+				(font
+					(size 1.27 1.27)
+				)
+			)
+		)
+		(property "Value" "GND"
+			(at 755.65 135.8899 90)
+			(show_name no)
+			(do_not_autoplace no)
+			(effects
+				(font
+					(size 1.27 1.27)
+				)
+				(justify right)
+			)
+		)
+		(property "Footprint" ""
+			(at 751.84 135.89 0)
+			(hide yes)
+			(show_name no)
+			(do_not_autoplace no)
+			(effects
+				(font
+					(size 1.27 1.27)
+				)
+			)
+		)
+		(property "Datasheet" ""
+			(at 751.84 135.89 0)
+			(hide yes)
+			(show_name no)
+			(do_not_autoplace no)
+			(effects
+				(font
+					(size 1.27 1.27)
+				)
+			)
+		)
+		(property "Description" "Power symbol creates a global label with name \"GND\" , ground"
+			(at 751.84 135.89 0)
+			(hide yes)
+			(show_name no)
+			(do_not_autoplace no)
+			(effects
+				(font
+					(size 1.27 1.27)
+				)
+			)
+		)
+		(pin "1"
+		)
+		(instances
+			(project "uTari_kicad"
+				(path "/a349f05f-5568-4b84-b3fc-0198b55a1cf7"
+					(reference "#PWR01")
+					(unit 1)
+				)
+			)
+		)
+	)
+	(symbol
+		(lib_id "power:GND")
 		(at 49.53 293.37 180)
 		(unit 1)
@@
 	)
 	(symbol
+		(lib_id "power:GND")
+		(at 751.84 138.43 90)
+		(unit 1)
+		(body_style 1)
+		(exclude_from_sim no)
+		(in_bom yes)
+		(on_board yes)
+		(in_pos_files yes)
+		(dnp no)
+		(fields_autoplaced yes)
+		(property "Reference" "#PWR02"
+			(at 758.19 138.43 0)
+			(hide yes)
+			(show_name no)
+			(do_not_autoplace no)
+			(effects
+				(font
+					(size 1.27 1.27)
+				)
+			)
+		)
+		(property "Value" "GND"
+			(at 755.65 138.4299 90)
+			(show_name no)
+			(do_not_autoplace no)
+			(effects
+				(font
+					(size 1.27 1.27)
+				)
+				(justify right)
+			)
+		)
+		(property "Footprint" ""
+			(at 751.84 138.43 0)
+			(hide yes)
+			(show_name no)
+			(do_not_autoplace no)
+			(effects
+				(font
+					(size 1.27 1.27)
+				)
+			)
+		)
+		(property "Datasheet" ""
+			(at 751.84 138.43 0)
+			(hide yes)
+			(show_name no)
+			(do_not_autoplace no)
+			(effects
+				(font
+					(size 1.27 1.27)
+				)
+			)
+		)
+		(property "Description" "Power symbol creates a global label with name \"GND\" , ground"
+			(at 751.84 138.43 0)
+			(hide yes)
+			(show_name no)
+			(do_not_autoplace no)
+			(effects
+				(font
+					(size 1.27 1.27)
+				)
+			)
+		)
+		(pin "1"
+		)
+		(instances
+			(project "uTari_kicad"
+				(path "/a349f05f-5568-4b84-b3fc-0198b55a1cf7"
+					(reference "#PWR02")
+					(unit 1)
+				)
+			)
+		)
+	)
+	(symbol
 		(lib_id "Device:C_Small_US")
 		(at 49.53 295.91 0)
@@
 			)
 		)
-		(property "Footprint" "Button_Switch_THT:SW_Slide-03_Wuerth-WS-SLTV_10x2.5x6.4_P2.54mm"
+		(property "Footprint" "Connector_PinHeader_2.54mm:PinHeader_1x03_P2.54mm_Vertical"
 			(at 39.37 292.1 0)
 			(hide yes)
@@
 			)
 		)
-		(property "Footprint" "Button_Switch_THT:SW_Slide-03_Wuerth-WS-SLTV_10x2.5x6.4_P2.54mm"
+		(property "Footprint" "Connector_PinHeader_2.54mm:PinHeader_1x03_P2.54mm_Vertical"
 			(at 81.28 535.94 0)
 			(hide yes)
@@
 	)
 	(symbol
+		(lib_id "Connector:Conn_01x02_Pin")
+		(at 746.76 135.89 0)
+		(unit 1)
+		(body_style 1)
+		(exclude_from_sim no)
+		(in_bom yes)
+		(on_board yes)
+		(in_pos_files yes)
+		(dnp no)
+		(fields_autoplaced yes)
+		(property "Reference" "J9"
+			(at 747.395 130.81 0)
+			(show_name no)
+			(do_not_autoplace no)
+			(effects
+				(font
+					(size 1.27 1.27)
+				)
+			)
+		)
+		(property "Value" "Ground Out"
+			(at 747.395 133.35 0)
+			(show_name no)
+			(do_not_autoplace no)
+			(effects
+				(font
+					(size 1.27 1.27)
+				)
+			)
+		)
+		(property "Footprint" "Connector_PinSocket_2.54mm:PinSocket_1x02_P2.54mm_Vertical"
+			(at 746.76 135.89 0)
+			(hide yes)
+			(show_name no)
+			(do_not_autoplace no)
+			(effects
+				(font
+					(size 1.27 1.27)
+				)
+			)
+		)
+		(property "Datasheet" ""
+			(at 746.76 135.89 0)
+			(hide yes)
+			(show_name no)
+			(do_not_autoplace no)
+			(effects
+				(font
+					(size 1.27 1.27)
+				)
+			)
+		)
+		(property "Description" "Generic connector, single row, 01x02, script generated"
+			(at 746.76 135.89 0)
+			(hide yes)
+			(show_name no)
+			(do_not_autoplace no)
+			(effects
+				(font
+					(size 1.27 1.27)
+				)
+			)
+		)
+		(pin "1"
+		)
+		(pin "2"
+		)
+		(instances
+			(project "uTari_kicad"
+				(path "/a349f05f-5568-4b84-b3fc-0198b55a1cf7"
+					(reference "J9")
+					(unit 1)
+				)
+			)
+		)
+	)
+	(symbol
 		(lib_id "Device:R")
 		(at 643.89 339.09 0)
@@
 			)
 		)
-		(property "Footprint" "Button_Switch_THT:SW_Slide-03_Wuerth-WS-SLTV_10x2.5x6.4_P2.54mm"
+		(property "Footprint" "Connector_PinHeader_2.54mm:PinHeader_1x03_P2.54mm_Vertical"
 			(at 39.37 325.12 0)
 			(hide yes)

Commit message: Minor board updates.
Parts:
- R27: value 2.2K -> 3.3K
- R28: value 1.6K -> 2.2K
- SW5: value Select -> Reset
- SW6: value Reset -> Select
Changed lines of the file:
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@@
 			)
 		)
-		(property "Value" "Select"
+		(property "Value" "Reset"
 			(at 39.37 336.55 0)
 			(show_name no)
@@
 			)
 		)
-		(property "Value" "1.6K"
+		(property "Value" "2.2K"
 			(at 777.24 223.5199 0)
 			(show_name no)
@@
 			)
 		)
-		(property "Value" "2.2K"
+		(property "Value" "3.3K"
 			(at 764.54 232.4099 0)
 			(show_name no)
@@
 			)
 		)
-		(property "Value" "Reset"
+		(property "Value" "Select"
 			(at 39.37 347.98 0)
 			(show_name no)
